File: Eagle/Main board/Main board.brd (EAGLE design)
At the start: 160 x 160 mm, 99 parts, among them IC1 LMZ14202TZE-ADJ_NOPB, IC2 VNH7070ASTR, IC3 VNH7070ASTR, IC4 VNH7070ASTR, IC5 VNH7070ASTR, J2 10104111-0001LF, SW1 TL38PO, SW2 TL38PO

Commit message: Added motor connectors, added electrolytic cap on supply
Parts:
- added C22: 100n, rcl:C0805
- added C23: EEV-FK1C152Q, Panasonic 1500uF:FKV(H13)
- added J3, J4, J5, J6: 43650-0201, Molex motori:43650-0200
- C1: value 10u -> 1500u
- C2: value 1u -> 100n
- C3: value 1u -> 10n
- C4: value 10u -> 22n
- C5: value 1u -> 100u; device rcl:C0805 -> rcl:C1206
- C6: value 1u -> 100u
- R3: value (none) -> 61,9k
- R4: value (none) -> 3,32k
- R5: value (none) -> 1,07k
- moved IC1 135.8 mm to (15.2, -41.9)
- moved U$2 57.0 mm to (36.2, -17.8), turned to 90 degrees
- moved J1 30.9 mm to (0.00, -54.9), flipped to the bottom
- moved U$4 8.89 mm to (13.3, -10.2)
- moved U$1 5.24 mm to (0.00, 43.2)
Connections:
- removed net VBAT-: J1.-, S_ELETTR..3, S_MOT.3
- net +12V: now also C23.1
- net +3V3: now also C22.1
- net GND: now also J1.-, S_ELETTR..3, S_MOT.3
- net M1_OUTA: now also J3.1
- net M1_OUTB: now also J3.2
- net M2_OUTA: now also J4.1
- net M2_OUTB: now also J4.2
- net M3_OUTA: now also J5.1
- net M3_OUTB: now also J5.2
- net M4_OUTA: now also J6.1
- net M4_OUTB: now also J6.2
- net N$4: now also C22.2, C23.2

Commit message: Added every component in BoM
Parts:
- added C25: 100n, rcl:C0805
- C1: value 1500u -> 100n
- C11, C12, C9: value (none) -> 100u
- C3: value 10n -> 22n
- C7: value (none) -> 1OOu
- RB1, RB2, RB3, RB4: value 33 -> 22
- moved J6 259.6 mm to (-53.6, -15.2), flipped to the bottom
- moved J3 254.9 mm to (-50.5, 15.2), flipped to the bottom, turned to 180 degrees
- moved J4 245.7 mm to (-37.8, 15.2), flipped to the bottom, turned to 180 degrees
- moved J5 244.4 mm to (-40.9, -15.2), flipped to the bottom
- moved IC4 222.7 mm to (-39.4, -7.62), turned to 270 degrees
- moved IC5 221.5 mm to (-52.1, -7.62), turned to 270 degrees
- moved IC2 177.4 mm to (-52.1, 7.62), turned to 90 degrees
- moved IC3 154.6 mm to (-39.4, 7.62), turned to 90 degrees
- moved S_ELETTR. 5.08 mm to (12.7, -58.4)
- moved S_MOT 5.08 mm to (-12.7, -58.4)
- renumbered CX to C24, SW1L1 to L1, SW2L1 to L2, SW2L2 to L3
Connections:
- net +3V3: now also C25.1
- net GND: now also C25.2
Routing:
- added copper zone on layer 1, net GND
- added copper zone on layer 16, net GND
- added copper zone on layer 1, net VBAT+
- added copper zone on layer 16, net VBAT+
- added copper zone on layer 1, net VMOT
- added copper zone on layer 16, net VMOT

Commit message: BoM finished
Parts:
- renumbered U$3 to IC6
Changed lines of the file:
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@@
 <element name="U$1" library="Teensy356" package="TEENSY_3.5/3.6" value="TEENSY_3.5/3.6" x="0" y="43.18" smashed="yes"/>
 <element name="U$2" library="OpenMV" package="OPENMV_H7" value="OPENMV_H7" x="36.19" y="-17.782" smashed="yes" rot="R90"/>
-<element name="U$3" library="Adafruit" package="TQFP44" value="ATMEGA32U4-AU" x="97.79" y="-7.62" smashed="yes">
+<element name="IC6" library="Adafruit" package="TQFP44" value="ATMEGA32U4-AU" x="97.79" y="-7.62" smashed="yes">
 <attribute name="NAME" x="93.98" y="-0.635" size="1.778" layer="25"/>
 <attribute name="VALUE" x="93.345" y="-16.3751" size="1.778" layer="27"/>
@@
 <contactref element="U$2" pad="3V3"/>
 <contactref element="C15" pad="1"/>
-<contactref element="U$3" pad="14"/>
-<contactref element="U$3" pad="44"/>
-<contactref element="U$3" pad="34"/>
-<contactref element="U$3" pad="24"/>
+<contactref element="IC6" pad="14"/>
+<contactref element="IC6" pad="44"/>
+<contactref element="IC6" pad="34"/>
+<contactref element="IC6" pad="24"/>
 <contactref element="R8" pad="2"/>
 <contactref element="C19" pad="1"/>
@@
 <contactref element="J2" pad="7"/>
 <contactref element="RST" pad="2"/>
-<contactref element="U$3" pad="5"/>
-<contactref element="U$3" pad="43"/>
+<contactref element="IC6" pad="5"/>
+<contactref element="IC6" pad="43"/>
 <contactref element="C16" pad="2"/>
 <contactref element="C17" pad="2"/>
 <contactref element="C18" pad="2"/>
-<contactref element="U$3" pad="15"/>
-<contactref element="U$3" pad="23"/>
-<contactref element="U$3" pad="35"/>
+<contactref element="IC6" pad="15"/>
+<contactref element="IC6" pad="23"/>
+<contactref element="IC6" pad="35"/>
 <contactref element="J2" pad="5"/>
 <contactref element="C20" pad="2"/>
@@
 <signal name="SP3">
 <contactref element="S3" pad="1"/>
-<contactref element="U$3" pad="25"/>
+<contactref element="IC6" pad="25"/>
 <wire x1="103.59" y1="-10.02" x2="51.28995" y2="54.88205" width="0" layer="19" extent="1-1"/>
 </signal>
 <signal name="SP4">
 <contactref element="S4" pad="1"/>
-<contactref element="U$3" pad="22"/>
+<contactref element="IC6" pad="22"/>
 <wire x1="101.79" y1="-13.42" x2="68.369984375" y2="31.048653125" width="0" layer="19" extent="1-1"/>
 </signal>
@@
 <signal name="SP1">
 <contactref element="S1" pad="1"/>
-<contactref element="U$3" pad="20"/>
+<contactref element="IC6" pad="20"/>
 <wire x1="-2.54" y1="74.93" x2="100.19" y2="-13.42" width="0" layer="19" extent="1-1"/>
 </signal>
 <signal name="SP2">
 <contactref element="S2" pad="1"/>
-<contactref element="U$3" pad="21"/>
+<contactref element="IC6" pad="21"/>
 <wire x1="100.99" y1="-13.42" x2="26.355346875" y2="70.314015625" width="0" layer="19" extent="1-1"/>
 </signal>
@@
 <signal name="SP5">
 <contactref element="S7" pad="1"/>
-<contactref element="U$3" pad="26"/>
+<contactref element="IC6" pad="26"/>
 <wire x1="54.882053125" y1="-51.289946875" x2="103.59" y2="-9.22" width="0" layer="19" extent="1-1"/>
 </signal>
 <signal name="SP6">
 <contactref element="S8" pad="1"/>
-<contactref element="U$3" pad="27"/>
+<contactref element="IC6" pad="27"/>
 <wire x1="31.04865625" y1="-68.36998125" x2="103.59" y2="-8.42" width="0" layer="19" extent="1-1"/>
 </signal>
 <signal name="SP7">
 <contactref element="S5" pad="1"/>
-<contactref element="U$3" pad="28"/>
+<contactref element="IC6" pad="28"/>
 <wire x1="74.93" y1="2.54" x2="103.59" y2="-7.62" width="0" layer="19" extent="1-1"/>
 </signal>
 <signal name="SP8">
 <contactref element="S6" pad="1"/>
-<contactref element="U$3" pad="29"/>
+<contactref element="IC6" pad="29"/>
 <wire x1="70.31401875" y1="-26.35534375" x2="103.59" y2="-6.82" width="0" layer="19" extent="1-1"/>
 </signal>
 <signal name="SP9">
 <contactref element="S11" pad="1"/>
-<contactref element="U$3" pad="30"/>
+<contactref element="IC6" pad="30"/>
 <wire x1="103.59" y1="-6.02" x2="-51.28995" y2="-54.88205" width="0" layer="19" extent="1-1"/>
 </signal>
 <signal name="SP10">
 <contactref element="S12" pad="1"/>
-<contactref element="U$3" pad="32"/>
+<contactref element="IC6" pad="32"/>
 <wire x1="-68.369984375" y1="-31.048653125" x2="103.59" y2="-4.42" width="0" layer="19" extent="1-1"/>
 </signal>
 <signal name="SP11">
 <contactref element="S9" pad="1"/>
-<contactref element="U$3" pad="31"/>
+<contactref element="IC6" pad="31"/>
 <wire x1="2.54" y1="-74.93" x2="103.59" y2="-5.22" width="0" layer="19" extent="1-1"/>
 </signal>
 <signal name="SP12">
 <contactref element="S10" pad="1"/>
-<contactref element="U$3" pad="36"/>
+<contactref element="IC6" pad="36"/>
 <wire x1="-26.355346875" y1="-70.314015625" x2="100.19" y2="-1.82" width="0" layer="19" extent="1-1"/>
 </signal>
 <signal name="SP13">
 <contactref element="S15" pad="1"/>
-<contactref element="U$3" pad="37"/>
+<contactref element="IC6" pad="37"/>
 <wire x1="-54.882053125" y1="51.289946875" x2="99.39" y2="-1.82" width="0" layer="19" extent="1-1"/>
 </signal>
 <signal name="SP14">
 <contactref element="S16" pad="1"/>
-<contactref element="U$3" pad="38"/>
+<contactref element="IC6" pad="38"/>
 <wire x1="-31.04865625" y1="68.36998125" x2="98.59" y2="-1.82" width="0" layer="19" extent="1-1"/>
 </signal>
 <signal name="SP15">
 <contactref element="S13" pad="1"/>
-<contactref element="U$3" pad="39"/>
+<contactref element="IC6" pad="39"/>
 <wire x1="-74.93" y1="-2.54" x2="97.79" y2="-1.82" width="0" layer="19" extent="1-1"/>
 </signal>
 <signal name="SP16">
 <contactref element="S14" pad="1"/>
-<contactref element="U$3" pad="40"/>
+<contactref element="IC6" pad="40"/>
 <wire x1="-70.31401875" y1="26.35534375" x2="96.99" y2="-1.82" width="0" layer="19" extent="1-1"/>
 </signal>
@@
 <signal name="N$5">
 <contactref element="C17" pad="1"/>
-<contactref element="U$3" pad="17"/>
+<contactref element="IC6" pad="17"/>
 <contactref element="Q1" pad="2"/>
 <wire x1="97.79" y1="-13.42" x2="113.35" y2="-29.21" width="0" layer="19" extent="1-1"/>
@@
 <signal name="N$6">
 <contactref element="C16" pad="1"/>
-<contactref element="U$3" pad="16"/>
+<contactref element="IC6" pad="16"/>
 <contactref element="Q1" pad="1"/>
 <wire x1="120.904" y1="-53.34" x2="118.43" y2="-29.21" width="0" layer="19" extent="1-1"/>
@@
 </signal>
 <signal name="N$7">
-<contactref element="U$3" pad="6"/>
+<contactref element="IC6" pad="6"/>
 <contactref element="C18" pad="1"/>
 <wire x1="108.27" y1="-29.21" x2="91.99" y2="-7.62" width="0" layer="19" extent="1-1"/>
@@
 <signal name="N$8">
 <contactref element="R6" pad="1"/>
-<contactref element="U$3" pad="3"/>
+<contactref element="IC6" pad="3"/>
 <wire x1="85.41" y1="-24.13" x2="91.99" y2="-5.22" width="0" layer="19" extent="1-1"/>
 </signal>
 <signal name="N$11">
 <contactref element="R7" pad="1"/>
-<contactref element="U$3" pad="4"/>
+<contactref element="IC6" pad="4"/>
 <wire x1="91.99" y1="-6.02" x2="180.66" y2="-17.78" width="0" layer="19" extent="1-1"/>
 </signal>
 <signal name="N$12">
 <contactref element="J2" pad="1"/>
-<contactref element="U$3" pad="7"/>
-<contactref element="U$3" pad="2"/>
+<contactref element="IC6" pad="7"/>
+<contactref element="IC6" pad="2"/>
 <wire x1="91.99" y1="-8.42" x2="91.99" y2="-4.42" width="0" layer="19" extent="1-1"/>
 <wire x1="104.11" y1="-62.31" x2="91.99" y2="-8.42" width="0" layer="19" extent="1-1"/>
 </signal>
 <signal name="MISO">
-<contactref element="U$3" pad="11"/>
+<contactref element="IC6" pad="11"/>
 <contactref element="J_SPI" pad="1"/>
 <wire x1="110.49" y1="-54.61" x2="91.99" y2="-11.62" width="0" layer="19" extent="1-1"/>
 </signal>
 <signal name="MOSI">
-<contactref element="U$3" pad="10"/>
+<contactref element="IC6" pad="10"/>
 <contactref element="J_SPI" pad="4"/>
 <wire x1="113.03" y1="-52.07" x2="91.99" y2="-10.82" width="0" layer="19" extent="1-1"/>
 </signal>
 <signal name="SCK">
-<contactref element="U$3" pad="9"/>
+<contactref element="IC6" pad="9"/>
 <contactref element="J_SPI" pad="3"/>
 <wire x1="113.03" y1="-54.61" x2="91.99" y2="-10.02" width="0" layer="19" extent="1-1"/>
@@
 <contactref element="J_SPI" pad="5"/>
 <contactref element="RST" pad="1"/>
-<contactref element="U$3" pad="13"/>
+<contactref element="IC6" pad="13"/>
 <contactref element="R8" pad="1"/>
 <wire x1="159.06" y1="-16.51" x2="175.58" y2="-17.78" width="0" layer="19" extent="1-1"/>

Commit message: Supply planes for motor drivers done
Parts:
- added U$3: BLUESMIRF, BlueSMIRF Silver:BLUESMIRF
- C19, C25, C6: device rcl:C0805 -> rcl:C1206
- CB1, CB2, CB3, CB4: device rcl:C1206 -> rcl:C0805
- moved C8 219.6 mm to (-61.6, 5.08), turned to 90 degrees
- moved C11 208.9 mm to (-67.3, 6.35), turned to 270 degrees
- moved C10 202.7 mm to (-61.6, -5.08), turned to 270 degrees
- moved C12 195.2 mm to (-67.3, -6.35), turned to 90 degrees
- moved C7 192.1 mm to (-28.6, 7.62), turned to 270 degrees
- moved C9 174.5 mm to (-19.7, 7.62), turned to 270 degrees
- moved C13 171.3 mm to (-34.9, -5.08), turned to 270 degrees
- moved C14 168.0 mm to (-34.9, 5.08), turned to 90 degrees
- moved J4 2.54 mm to (-40.4, 15.2)
- moved IC2 2.54 mm to (-54.6, 7.62)
- moved IC3 2.54 mm to (-41.9, 7.62)
- moved IC4 2.54 mm to (-41.9, -7.62)
- moved IC5 2.54 mm to (-54.6, -7.62)
- moved J3 2.54 mm to (-53.1, 15.2)
- moved J5 2.54 mm to (-43.4, -15.2)
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Connections:
- net +3V3: now also U$3.VCC
- net GND: now also U$3.GND
- net M1_OUTA: now also J3.2; no longer J3.1
- net M1_OUTB: now also J3.1; no longer J3.2
- net M2_OUTA: now also J4.2; no longer J4.1
- net M2_OUTB: now also J4.1; no longer J4.2
- net M3_OUTA: now also J5.2; no longer J5.1
- net M3_OUTB: now also J5.1; no longer J5.2
- net M4_OUTA: now also J6.2; no longer J6.1
- net M4_OUTB: now also J6.1; no longer J6.2
- net RX3: now also U$3.TX
- net TX3: now also U$3.RX
