File: Eagle/Main board/Main board.brd (EAGLE design)
At the start: 160 x 160 mm, 108 parts, among them IC1 LMZ14202TZE-ADJ_NOPB, IC2 VNH7070ASTR, IC3 VNH7070ASTR, IC4 VNH7070ASTR, IC5 VNH7070ASTR, IC6 ATMEGA32U4-AU, J2 10104111-0001LF, J3 43650-0201, J4 43650-0201, J5 43650-0201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

Commit message: PCB layout almost done
Parts:
- removed M1_A, M1_C, M2_A, M2_C, M3_A, M3_C, M4_A, M4_C: (no value), led:CHIPLED_1206
- added L4, M1+, M1-, M2+, M2-, M3+, M3-, M4+, M4-: (no value), led:CHIPLED_1206
- added R18: (no value), rcl:R0805
- U$2: device OpenMV:OPENMV_H7 -> OpenMV4:OPENMV_H7
- moved U$3 90.3 mm to (-97.8, -22.9)
- moved C26 88.9 mm to (-133.3, -31.8)
- moved R11 70.0 mm to (-45.7, -31.8)
- moved R13 61.3 mm to (123.4, -38.6)
- moved R14 60.1 mm to (122.2, -30.0)
- moved L2 59.6 mm to (53.3, -22.1), turned to 180 degrees
- moved SW1L 59.0 mm to (117.3, -39.6)
- moved R12 58.8 mm to (-58.4, -31.8)
- moved SW2L 58.8 mm to (117.1, -29.5)
- moved SW2 57.4 mm to (106.9, -31.2)
- moved SW1 56.7 mm to (106.2, -39.4)
- moved L1 53.1 mm to (49.5, -22.1), turned to 180 degrees
- moved R16 51.1 mm to (53.3, -15.2), flipped to the bottom, turned to 270 degrees
- moved LS_SUD 47.8 mm to (21.0, 57.0), flipped to the bottom
- moved R15 46.6 mm to (49.5, -15.2), flipped to the bottom, turned to 270 degrees
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Connections:
- removed net POWER_BLOK_1: CB2.1, RB2.2, S5.3, S6.3, S7.3, S8.3
- removed net POWER_BLOK_2: CB1.1, RB1.2, S1.3, S2.3, S3.3, S4.3
- removed net POWER_BLOK_3: CB3.1, RB3.2, S10.3, S11.3, S12.3, S9.3
- removed net POWER_BLOK_4: CB4.1, RB4.2, S13.3, S14.3, S15.3, S16.3
- new net LED4: IC6.8, R18.1
- new net N$4: L4.A, R18.2
- new net POWER_BLOCK_1: CB1.1, RB1.2, S2.3, S3.3, S4.3, S5.3
- new net POWER_BLOCK_2: CB2.1, RB2.2, S6.3, S7.3, S8.3, S9.3
- new net POWER_BLOCK_3: CB3.1, RB3.2, S10.3, S11.3, S12.3, S13.3
- new net POWER_BLOCK_4: CB4.1, RB4.2, S1.3, S14.3, S15.3, S16.3
- net E_EST: now also U$1.33/A14; no longer U$1.34/A15
- net E_INT: now also U$1.34/A15; no longer U$1.33/A14
- net GND: now also L4.C
- net LED1: now also IC6.22; no longer U$1.14/A0
- net LED2: now also IC6.41; no longer U$1.15/A1
- net LED3: now also IC6.12; no longer U$1.16/A2
- net M1_INA: now also M1+.A; no longer M1_C.A
- net M1_INB: now also M1-.A; no longer M1_A.A
- net M1_PWM: now also U$1.4/CANRX; no longer U$1.2
- net M2_INA: now also M2+.A; no longer M2_C.A
- net M2_INB: now also M2-.A; no longer M2_A.A
- net M2_PWM: now also U$1.5; no longer U$1.3/CANTX
- net M3_INA: now also M3+.A; no longer M3_C.A
- net M3_INB: now also M3-.A; no longer M3_A.A
- net M3_PWM: now also U$1.2; no longer U$1.4/CANRX
- net M4_INA: now also M4+.A; no longer M4_C.A
- net M4_INB: now also M4-.A; no longer M4_A.A
- net M4_PWM: now also U$1.3/CANTX; no longer U$1.5
- net N$12: no longer IC6.2
- net N$13: now also M2+.C, M2-.C; no longer M2_A.C, M2_C.C
- net N$14: now also M1+.C, M1-.C; no longer M1_A.C, M1_C.C
- net N$15: now also M3+.C, M3-.C; no longer M3_A.C, M3_C.C
- net N$16: now also M4+.C, M4-.C; no longer M4_A.C, M4_C.C
- net N_EST: now also U$1.35/A16; no longer U$1.32/A13
- net N_INT: now also U$1.36/A17; no longer U$1.31/A12
- net O_EST: now also U$1.37/A18; no longer U$1.38/A19
- net O_INT: now also U$1.38/A19; no longer U$1.37/A18
- net RX1: now also U$3.TX
- net RX2: now also IC6.21; no longer U$2.P4
- net RX3: now also U$2.P4; no longer U$3.TX
- net SP1: now also IC6.26; no longer IC6.20
- net SP10: now also IC6.36, S10.1; no longer IC6.32, S12.1
- net SP11: now also IC6.32, S11.1; no longer IC6.31, S9.1
- net SP12: now also IC6.31, S12.1; no longer IC6.36, S10.1
- net SP13: now also IC6.30, S13.1; no longer IC6.37, S15.1
- net SP14: now also IC6.29, S14.1; no longer IC6.38, S16.1
- net SP15: now also IC6.28, S15.1; no longer IC6.39, S13.1
- net SP16: now also IC6.27, S16.1; no longer IC6.40, S14.1
- net SP2: now also IC6.25; no longer IC6.21
- net SP3: now also IC6.19; no longer IC6.25
- net SP4: now also IC6.18; no longer IC6.22
- net SP5: now also IC6.1, S5.1; no longer IC6.26, S7.1
- net SP6: now also IC6.40, S6.1; no longer IC6.27, S8.1
- net SP7: now also IC6.39, S7.1; no longer IC6.28, S5.1
- net SP8: now also IC6.38, S8.1; no longer IC6.29, S6.1
- net SP9: now also IC6.37, S9.1; no longer IC6.30, S11.1
- net S_EST: now also U$1.32/A13; no longer U$1.36/A17
- net S_INT: now also U$1.31/A12; no longer U$1.35/A16
- net TX1: now also U$3.RX
- net TX2: now also IC6.20; no longer U$2.P5
- net TX3: now also U$2.P5; no longer U$3.RX
Routing:
- net SP11: track 0.00 -> 289.9 mm
- net SP12: track 0.00 -> 260.4 mm
- net SP13: track 0.00 -> 231.0 mm
- net SP14: track 0.00 -> 202.3 mm
- net SP15: track 0.00 -> 171.1 mm
- net SP10: track 0.00 -> 140.3 mm
- net SP16: track 0.00 -> 140.3 mm
- net M4_INB: track 0.00 -> 139.0 mm, vias 0 -> 4
- net M4_INA: track 0.00 -> 130.8 mm, vias 0 -> 6
- net M4_PWM: track 0.00 -> 129.9 mm, vias 0 -> 1
- net M3_PWM: track 0.00 -> 128.4 mm, vias 0 -> 1
- net M3_INB: track 0.00 -> 122.9 mm, vias 0 -> 6
- net M3_INA: track 0.00 -> 119.3 mm, vias 0 -> 6
- net SP9: track 0.00 -> 113.7 mm
- net SP1: track 0.00 -> 110.2 mm
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- added copper zone on layer 16, net GND3
- added copper zone on layer 1, net POWER_BLOCK_1
- added copper zone on layer 1, net POWER_BLOCK_2
- added copper zone on layer 1, net POWER_BLOCK_3
- added copper zone on layer 1, net POWER_BLOCK_4

Commit message: PCB almost done
Parts:
- removed U$3: BLUESMIRF, BlueSMIRF Silver:BLUESMIRF
- added BLUETOOTH: TWIG_2.0, CONNECTER:2.0_1X4
- moved CB2 171.2 mm to (59.7, -34.3), turned to 180 degrees
- moved RB2 168.2 mm to (59.7, -31.8)
- moved C26 130.7 mm to (-33.0, 52.1), turned to 180 degrees
- moved CB3 130.1 mm to (-35.6, -64.8)
- moved RB1 127.3 mm to (44.5, 55.9)
- moved CB1 127.2 mm to (44.5, 58.4), turned to 180 degrees
- moved RB3 124.5 mm to (-35.6, -62.2), turned to 180 degrees
- moved RB4 113.4 mm to (7.62, 77.5), turned to 180 degrees
- moved BUZZER 112.1 mm to (26.0, 0.00)
- moved CB4 111.9 mm to (7.62, 74.9)
- moved R13 96.7 mm to (52.7, 27.3), flipped to the bottom, turned to 180 degrees
- moved SW1L 94.4 mm to (50.8, 27.3), turned to 90 degrees
- moved SW1 92.2 mm to (50.8, 34.3), turned to 270 degrees
- moved R14 85.2 mm to (59.1, 27.3), flipped to the bottom, turned to 180 degrees
- moved SW2L 82.6 mm to (57.1, 27.3), turned to 90 degrees
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Connections:
- net +3V3: now also BLUETOOTH.1; no longer U$3.VCC
- net GND: now also BLUETOOTH.2, R13.2, R14.2; no longer SW1L.C, SW2L.C, U$3.GND
- net N$17: now also R13.1, SW1L.C; no longer R14.2, SW2L.A
- net N$18: now also R14.1, SW2L.C; no longer R13.2, SW1L.A
- net RX1: now also BLUETOOTH.3; no longer U$3.TX
- net SW1: now also SW1L.A; no longer R13.1
- net SW2: now also SW2L.A; no longer R14.1
- net TX1: now also BLUETOOTH.4; no longer U$3.RX
Routing:
- net +3V3: track 89.7 -> 575.0 mm, vias 0 -> 5
- net SW1: track 0.00 -> 97.6 mm, vias 0 -> 1
- net SW2: track 0.00 -> 95.9 mm, vias 0 -> 1
- net SCL: track 0.00 -> 67.8 mm, vias 0 -> 1
- net SDA: track 0.00 -> 65.2 mm, vias 0 -> 1
- net BUZZ: track 0.00 -> 49.0 mm, vias 0 -> 1
- net TX1: track 0.00 -> 36.2 mm
- net RX1: track 0.00 -> 25.8 mm
- net POWER_BLOCK_2: track 0.00 -> 23.8 mm, vias 0 -> 2
- net RST: track 0.00 -> 23.4 mm, vias 0 -> 1
- net POWER_BLOCK_3: track 0.00 -> 19.4 mm
- net POWER_BLOCK_1: track 0.00 -> 19.4 mm
- net POWER_BLOCK_4: track 0.00 -> 18.1 mm
- net +12V: track 41.9 -> 46.0 mm
- net GND: track 35.5 -> 38.3 mm
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