File: Eagle/Main board/Main board.sch (EAGLE design)
At the start: 108 parts, among them IC1 LMZ14202TZE-ADJ_NOPB, IC2 VNH7070ASTR, IC3 VNH7070ASTR, IC4 VNH7070ASTR, IC5 VNH7070ASTR, IC6 ATMEGA32U4-AU, J2 10104111-0001LF, J3 43650-0201, J4 43650-0201, J5 43650-0201, J6 43650-0201, SW1 TL38PO, SW2 TL38PO

Commit message: PCB layout almost done
Parts:
- added L4: (no value), led:LEDCHIPLED_1206
- added R18: (no value), rcl:R-EU_R0805
- U$2: device OpenMV:OPENMV_H7 -> OpenMV4:OPENMV_H7
- renumbered M1_A to M1-, M1_C to M1+, M2_A to M2-, M2_C to M2+, M3_A to M3-, M3_C to M3+, M4_A to M4-, M4_C to M4+
Connections:
- removed net POWER_BLOK_1: CB2.1, RB2.2, S5.VCC, S6.VCC, S7.VCC, S8.VCC
- removed net POWER_BLOK_2: CB1.1, RB1.2, S1.VCC, S2.VCC, S3.VCC, S4.VCC
- removed net POWER_BLOK_3: CB3.1, RB3.2, S10.VCC, S11.VCC, S12.VCC, S9.VCC
- removed net POWER_BLOK_4: CB4.1, RB4.2, S13.VCC, S14.VCC, S15.VCC, S16.VCC
- new net LED4: IC6.PB0(SS), R18.1
- new net N$4: L4.A, R18.2
- new net POWER_BLOCK_1: CB1.1, RB1.2, S2.VCC, S3.VCC, S4.VCC, S5.VCC
- new net POWER_BLOCK_2: CB2.1, RB2.2, S6.VCC, S7.VCC, S8.VCC, S9.VCC
- new net POWER_BLOCK_3: CB3.1, RB3.2, S10.VCC, S11.VCC, S12.VCC, S13.VCC
- new net POWER_BLOCK_4: CB4.1, RB4.2, S1.VCC, S14.VCC, S15.VCC, S16.VCC
- net E_EST: now also U$1.33/A14; no longer U$1.34/A15
- net E_INT: now also U$1.34/A15; no longer U$1.33/A14
- net GND: now also L4.C
- net LED1: now also IC6.PD5(XCK/CTS); no longer U$1.14/A0
- net LED2: now also IC6.PF0(ADC0); no longer U$1.15/A1
- net LED3: now also IC6.PB7(OC0A/OC1C/RTS); no longer U$1.16/A2
- net M1_PWM: now also U$1.4/CANRX; no longer U$1.2
- net M2_PWM: now also U$1.5; no longer U$1.3/CANTX
- net M3_PWM: now also U$1.2; no longer U$1.4/CANRX
- net M4_PWM: now also U$1.3/CANTX; no longer U$1.5
- net N$12: no longer IC6.UVCC
- net N_EST: now also U$1.35/A16; no longer U$1.32/A13
- net N_INT: now also U$1.36/A17; no longer U$1.31/A12
- net O_EST: now also U$1.37/A18; no longer U$1.38/A19
- net O_INT: now also U$1.38/A19; no longer U$1.37/A18
- net RX1: now also U$3.TX
- net RX2: now also IC6.PD3(INT3/TXD1); no longer U$2.P4
- net RX3: now also U$2.P4; no longer U$3.TX
- net SP1: now also IC6.PD6(T1/ADC9/!OC4D); no longer IC6.PD2(INT2/RXD1)
- net SP10: now also IC6.PF7(ADC7(TDI), S10.OUT; no longer IC6.PC7(ICP3/CLK0/OC4A), S12.OUT
- net SP11: now also IC6.PC7(ICP3/CLK0/OC4A), S11.OUT; no longer IC6.PC6(OC3A/!OC4A), S9.OUT
- net SP12: now also IC6.PC6(OC3A/!OC4A), S12.OUT; no longer IC6.PF7(ADC7(TDI), S10.OUT
- net SP13: now also IC6.PB6(OC1B/OC4B/ADC13), S13.OUT; no longer IC6.PF6(ADC6/TDO), S15.OUT
- net SP14: now also IC6.PB5(OC1A/ADC12/!OC4B), S14.OUT; no longer IC6.PF5(ADC5/TMS), S16.OUT
- net SP15: now also IC6.PB4(ADC11), S15.OUT; no longer IC6.PF4(ADC4/TCK), S13.OUT
- net SP16: now also IC6.PD7(OC4D/ADC10/T0), S16.OUT; no longer IC6.PF1(ADC1), S14.OUT
- net SP2: now also IC6.PD4(ICP1/ADC8); no longer IC6.PD3(INT3/TXD1)
- net SP3: now also IC6.PD1(INT1/SDA); no longer IC6.PD4(ICP1/ADC8)
- net SP4: now also IC6.PD0(INT0/OC0B/SCL); no longer IC6.PD5(XCK/CTS)
- net SP5: now also IC6.PE6(INT.6/AIN0), S5.OUT; no longer IC6.PD6(T1/ADC9/!OC4D), S7.OUT
- net SP6: now also IC6.PF1(ADC1), S6.OUT; no longer IC6.PD7(OC4D/ADC10/T0), S8.OUT
- net SP7: now also IC6.PF4(ADC4/TCK), S7.OUT; no longer IC6.PB4(ADC11), S5.OUT
- net SP8: now also IC6.PF5(ADC5/TMS), S8.OUT; no longer IC6.PB5(OC1A/ADC12/!OC4B), S6.OUT
- net SP9: now also IC6.PF6(ADC6/TDO), S9.OUT; no longer IC6.PB6(OC1B/OC4B/ADC13), S11.OUT
- net S_EST: now also U$1.32/A13; no longer U$1.36/A17
- net S_INT: now also U$1.31/A12; no longer U$1.35/A16
- net TX1: now also U$3.RX
- net TX2: now also IC6.PD2(INT2/RXD1); no longer U$2.P5
- net TX3: now also U$2.P5; no longer U$3.RX
Other:
- moved on the sheet: L1, L2, L3, R15, R16, R17, S1, S10, S11, S12, S13, S14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

Commit message: PCB almost done
Parts:
- removed U$3: BLUESMIRF, BlueSMIRF Silver:BLUESMIRF
- added BLUETOOTH: TWIG_2.0, CONNECTER:TWIG_2.0
Connections:
- net +3V3: now also BLUETOOTH.1; no longer U$3.VCC
- net GND: now also BLUETOOTH.2, R13.2, R14.2; no longer SW1L.C, SW2L.C, U$3.GND
- net N$17: now also R13.1, SW1L.C; no longer R14.2, SW2L.A
- net N$18: now also R14.1, SW2L.C; no longer R13.2, SW1L.A
- net RX1: now also BLUETOOTH.3; no longer U$3.TX
- net SW1: now also SW1L.A; no longer R13.1
- net SW2: now also SW2L.A; no longer R14.1
- net TX1: now also BLUETOOTH.4; no longer U$3.RX
Other:
- moved on the sheet: C26, J_SPI, R13, R14, SW1L, SW2L
