File: Eagle/Main board/Main board.sch (EAGLE design)
At the start: 123 parts, among them IC1 LMZ14202TZE-ADJ_NOPB, IC2 VNH7070ASTR, IC3 VNH7070ASTR, IC4 VNH7070ASTR, IC5 VNH7070ASTR, IC6 ATMEGA32U4-AU, J3 43650-0201, J4 43650-0201, J5 43650-0201, J6 43650-0201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

Commit message: Added RCWL compatible ToF
Parts:
- added C27: 100n, rcl:C-EUC0805
- added R32: (no value), rcl:R-EU_R0805
- added SW3: TL38PO, switch:TL38PO
- added SW3L: (no value), led:LEDCHIPLED_1206
- added TOF: TWIG_2.0, CONNECTER:TWIG_2.0
- S_ELETTR., S_MOT: device switch:320-916 -> Switch:255SB
Connections:
- removed net BPS: U$1.39/A20
- removed net KICK: U$1.20/A6
- removed net ROLL: U$1.21/A7
- new net A/TRIG: TOF.2, U$1.35/A16
- new net ECHO: TOF.3, U$1.36/A17
- new net SW3: SW3.P, SW3L.A, U$1.37/A18
- net +3V3: now also C27.1, SW3.O, TOF.1
- net E_EST: now also U$1.16/A2; no longer U$1.33/A14
- net E_INT: now also U$1.17/A3; no longer U$1.34/A15
- net GND: now also C27.2, R32.2, SW3.S, TOF.4
- net N$19: now also R32.1, SW3L.C; no longer U$1.30
- net N_EST: now also U$1.20/A6; no longer U$1.35/A16
- net N_INT: now also U$1.21/A7; no longer U$1.36/A17
- net O_EST: now also U$1.22/A8; no longer U$1.37/A18
- net O_INT: now also U$1.23/A9; no longer U$1.38/A19
- net SW1: now also U$1.39/A20; no longer U$1.23/A9
- net SW2: now also U$1.38/A19; no longer U$1.22/A8
- net S_EST: now also U$1.14/A0; no longer U$1.32/A13
- net S_INT: now also U$1.15/A1; no longer U$1.31/A12
Other:
- note added: "ToF"
- moved on the sheet: C25, LD1, LD2, LD3, LD4, R15, R16, R17, R18

Commit message: Main board done
Parts:
- added BALL, MULTI1, MULTI2: TWIG_2.0, CONNECTER:TWIG_2.0
- added BAT, ELECT, MOT: (no value), led:LEDCHIPLED_1206
- added C28: EEV-FK1C152Q, Panasonic 1500uF:EEV-FK1C152Q
- added J2, J7: 43650-0201, Molex motori:43650-0201
- added R33, R34, R35: (no value), rcl:R-EU_R0805
Connections:
- new net BALL_IN: BALL.2, U$1.32/A13
- new net BALL_OUT: BALL.3, U$1.A22/DAC1
- new net MULTI_DIG1: MULTI1.3, U$1.31/A12
- new net MULTI_DIG2: MULTI2.3, U$1.34/A15
- new net MULTI_PWM1: MULTI1.2, U$1.30
- new net MULTI_PWM2: MULTI2.2, U$1.35/A16
- new net N$24: BAT.A, R33.2
- new net N$25: MOT.A, R34.2
- new net N$26: ELECT.A, R35.1
- net +3V3: now also BALL.1, MULTI1.1, MULTI2.1, R35.2
- net A/TRIG: now also U$1.36/A17; no longer U$1.35/A16
- net ECHO: now also U$1.37/A18; no longer U$1.36/A17
- net GND: now also BALL.4, BAT.C, ELECT.C, MOT.C, MULTI1.4, MULTI2.4
- net SW3: now also U$1.33/A14; no longer U$1.37/A18
- net V-: now also C28.-, J2.2, J7.2
- net VBAT+: now also R33.1
- net VMOT: now also C28.+, J2.1, J7.1, R34.1
Other:
- note added: "KICKER/MULTIPURPOSE"
- note added: "PALLA_PRESA"
- note added: "ROLLER/MULTIPURPOSE"
- moved on the sheet: BLUETOOTH, C24, C25, C26, C27, J3, J4, J5, J6, J_SPI, LD1, LD2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

Commit message: Job finished. Ready to print
Parts:
- removed R19: (no value), rcl:R-EU_R1206
- added TOF_TOP: TWIG_2.0, CONNECTER:TWIG_2.0
Connections:
- net +3V3: now also TOF_TOP.1
- net A/TRIG: now also TOF_TOP.2
- net ECHO: now also TOF_TOP.3
- net GND: now also TOF_TOP.4; no longer R19.2
- net V-: no longer R19.1
Changed lines of the file:
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@@
 <part name="P-9" library="supply1" library_urn="urn:adsk.eagle:library:371" deviceset="V-" device=""/>
 <part name="GND29" library="supply1" deviceset="GND" device=""/>
-<part name="R19" library="rcl" library_urn="urn:adsk.eagle:library:334" deviceset="R-EU_" device="R1206" package3d_urn="urn:adsk.eagle:package:23540/2"/>
 <part name="GND30" library="supply1" deviceset="GND" device=""/>
 <part name="GND31" library="supply1" deviceset="GND" device=""/>
@@
 <part name="C28" library="Panasonic 1500uF" deviceset="EEV-FK1C152Q" device=""/>
 <part name="P-12" library="supply1" library_urn="urn:adsk.eagle:library:371" deviceset="V-" device=""/>
+<part name="TOF_TOP" library="CONNECTER" deviceset="TWIG_2.0" device=""/>
 </parts>
 <sheets>
@@
 <wire x1="332.74" y1="132.08" x2="332.74" y2="162.56" width="0.1524" layer="97"/>
 <text x="358.14" y="129.54" size="1.778" layer="97" rot="MR0">BLUETOOTH</text>
-<wire x1="375.92" y1="185.42" x2="398.78" y2="185.42" width="0.1524" layer="97"/>
+<wire x1="363.22" y1="185.42" x2="398.78" y2="185.42" width="0.1524" layer="97"/>
 <wire x1="398.78" y1="185.42" x2="398.78" y2="162.56" width="0.1524" layer="97"/>
-<wire x1="398.78" y1="162.56" x2="375.92" y2="162.56" width="0.1524" layer="97"/>
-<wire x1="375.92" y1="162.56" x2="375.92" y2="185.42" width="0.1524" layer="97"/>
+<wire x1="398.78" y1="162.56" x2="363.22" y2="162.56" width="0.1524" layer="97"/>
+<wire x1="363.22" y1="162.56" x2="363.22" y2="185.42" width="0.1524" layer="97"/>
 <text x="398.78" y="160.02" size="1.778" layer="97" rot="MR0">ToF</text>
 <wire x1="-12.7" y1="261.62" x2="48.26" y2="261.62" width="0.1524" layer="97"/>
@@
 <attribute name="VALUE" x="91.44" y="135.89" size="1.778" layer="96"/>
 </instance>
-<instance part="R19" gate="G$1" x="85.09" y="142.24" smashed="yes">
-<attribute name="NAME" x="81.28" y="143.7386" size="1.778" layer="95"/>
-<attribute name="VALUE" x="81.28" y="138.938" size="1.778" layer="96"/>
-</instance>
 <instance part="GND30" gate="1" x="21.59" y="186.69" smashed="yes">
 <attribute name="VALUE" x="19.05" y="184.15" size="1.778" layer="96"/>
@@
 <attribute name="VALUE" x="271.78" y="144.78" size="1.778" layer="96" rot="R270"/>
 </instance>
+<instance part="TOF_TOP" gate="G$1" x="370.84" y="173.99" smashed="yes" rot="MR0">
+<attribute name="NAME" x="373.38" y="166.37" size="1.27" layer="95" rot="MR0"/>
+</instance>
 </instances>
 <busses>
@@
 <wire x1="384.81" y1="177.8" x2="388.62" y2="177.8" width="0.1524" layer="91"/>
 <wire x1="388.62" y1="177.8" x2="388.62" y2="179.07" width="0.1524" layer="91"/>
+<pinref part="TOF_TOP" gate="G$1" pin="1"/>
+<wire x1="374.65" y1="177.8" x2="384.81" y2="177.8" width="0.1524" layer="91"/>
+<junction x="384.81" y="177.8"/>
 </segment>
 <segment>
@@
 <wire x1="93.98" y1="140.97" x2="93.98" y2="142.24" width="0.1524" layer="91"/>
 <wire x1="93.98" y1="142.24" x2="90.17" y2="142.24" width="0.1524" layer="91"/>
-<pinref part="R19" gate="G$1" pin="2"/>
 </segment>
 <segment>
@@
 <wire x1="384.81" y1="170.18" x2="388.62" y2="170.18" width="0.1524" layer="91"/>
 <wire x1="388.62" y1="170.18" x2="388.62" y2="168.91" width="0.1524" layer="91"/>
+<pinref part="TOF_TOP" gate="G$1" pin="4"/>
+<wire x1="374.65" y1="170.18" x2="384.81" y2="170.18" width="0.1524" layer="91"/>
+<junction x="384.81" y="170.18"/>
 </segment>
 <segment>
@@
 <wire x1="76.2" y1="140.97" x2="76.2" y2="142.24" width="0.1524" layer="91"/>
 <wire x1="76.2" y1="142.24" x2="80.01" y2="142.24" width="0.1524" layer="91"/>
-<pinref part="R19" gate="G$1" pin="1"/>
 </segment>
 <segment>
@@
 <wire x1="384.81" y1="175.26" x2="396.24" y2="175.26" width="0.1524" layer="91"/>
 <label x="396.24" y="175.26" size="1.778" layer="95" rot="MR0"/>
+<pinref part="TOF_TOP" gate="G$1" pin="2"/>
+<wire x1="374.65" y1="175.26" x2="384.81" y2="175.26" width="0.1524" layer="91"/>
+<junction x="384.81" y="175.26"/>
 </segment>
 <segment>
@@
 <wire x1="384.81" y1="172.72" x2="396.24" y2="172.72" width="0.1524" layer="91"/>
 <label x="396.24" y="172.72" size="1.778" layer="95" rot="MR0"/>
+<pinref part="TOF_TOP" gate="G$1" pin="3"/>
+<wire x1="374.65" y1="172.72" x2="384.81" y2="172.72" width="0.1524" layer="91"/>
+<junction x="384.81" y="172.72"/>
 </segment>
 <segment>

Commit message: Final commit
Parts:
- renumbered ELECT to LD_ELECT
Changed lines of the file:
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@@
 <setting verticaltext="up"/>
 </settings>
-<grid distance="0.1" unitdist="inch" unit="inch" style="lines" multiple="1" display="yes" altdistance="0.05" altunitdist="inch" altunit="inch"/>
+<grid distance="0.1" unitdist="inch" unit="inch" style="lines" multiple="1" display="no" altdistance="0.01" altunitdist="inch" altunit="inch"/>
 <layers>
 <layer number="1" name="Top" color="4" fill="1" visible="no" active="no"/>
@@
 <part name="MOT" library="led" library_urn="urn:adsk.eagle:library:259" deviceset="LED" device="CHIPLED_1206" package3d_urn="urn:adsk.eagle:package:15823/2"/>
 <part name="R34" library="rcl" library_urn="urn:adsk.eagle:library:334" deviceset="R-EU_" device="R0805" package3d_urn="urn:adsk.eagle:package:23553/2"/>
-<part name="ELECT" library="led" library_urn="urn:adsk.eagle:library:259" deviceset="LED" device="CHIPLED_1206" package3d_urn="urn:adsk.eagle:package:15823/2"/>
+<part name="LD_ELECT" library="led" library_urn="urn:adsk.eagle:library:259" deviceset="LED" device="CHIPLED_1206" package3d_urn="urn:adsk.eagle:package:15823/2"/>
 <part name="R35" library="rcl" library_urn="urn:adsk.eagle:library:334" deviceset="R-EU_" device="R0805" package3d_urn="urn:adsk.eagle:package:23553/2"/>
 <part name="BALL" library="CONNECTER" deviceset="TWIG_2.0" device=""/>
@@
 <attribute name="VALUE" x="259.842" y="142.24" size="1.778" layer="96" rot="R90"/>
 </instance>
-<instance part="ELECT" gate="G$1" x="408.94" y="21.59" smashed="yes">
+<instance part="LD_ELECT" gate="G$1" x="408.94" y="21.59" smashed="yes">
 <attribute name="NAME" x="412.496" y="11.938" size="1.778" layer="95" rot="R90"/>
 <attribute name="VALUE" x="414.655" y="17.018" size="1.778" layer="96" rot="R90"/>
@@
 <wire x1="408.94" y1="12.7" x2="403.86" y2="12.7" width="0.1524" layer="91"/>
 <junction x="403.86" y="12.7"/>
-<pinref part="ELECT" gate="G$1" pin="C"/>
+<pinref part="LD_ELECT" gate="G$1" pin="C"/>
 <wire x1="408.94" y1="16.51" x2="408.94" y2="12.7" width="0.1524" layer="91"/>
 </segment>
@@
 <segment>
 <pinref part="R35" gate="G$1" pin="1"/>
-<pinref part="ELECT" gate="G$1" pin="A"/>
+<pinref part="LD_ELECT" gate="G$1" pin="A"/>
 <wire x1="408.94" y1="29.21" x2="408.94" y2="24.13" width="0.1524" layer="91"/>
 </segment>
