File: Eagle/Line sensors 2020/Line sensors - 4/Line sensors - 4.brd (EAGLE design)
At the start: 58.2 x 24.2 mm, 19 parts, among them Q1 VEMT2520X01, Q2 VEMT2520X01, Q3 VEMT2520X01, Q4 VEMT2520X01

Commit message: Final commit
Parts:
- removed CON: (no value), pinhead:1X04
- added MULTI2: TWIG_2.0, CONNECTER:2.0_1X4
Connections:
- net GND: now also MULTI2.4; no longer CON.4
- net SIG1: now also MULTI2.2; no longer CON.2
- net SIG2: now also MULTI2.3; no longer CON.3
- net V+: now also MULTI2.1; no longer CON.1
Changed lines of the file:
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@@
 <setting verticaltext="up"/>
 </settings>
-<grid distance="50" unitdist="mil" unit="mil" style="lines" multiple="1" display="yes" altdistance="25" altunitdist="mil" altunit="mil"/>
+<grid distance="10" unitdist="mil" unit="mil" style="lines" multiple="1" display="yes" altdistance="5" altunitdist="mil" altunit="mil"/>
 <layers>
 <layer number="1" name="Top" color="4" fill="1" visible="yes" active="yes"/>
@@
 <layer number="59" name="tCarbon" color="7" fill="1" visible="no" active="no"/>
 <layer number="60" name="bCarbon" color="7" fill="1" visible="no" active="no"/>
+<layer number="61" name="stand" color="7" fill="1" visible="no" active="no"/>
 <layer number="88" name="SimResults" color="9" fill="1" visible="no" active="no"/>
 <layer number="89" name="SimProbes" color="9" fill="1" visible="no" active="no"/>
@@
 <layer number="115" name="ReferenceISLANDS" color="7" fill="1" visible="no" active="yes"/>
 <layer number="116" name="Patch_BOT" color="9" fill="4" visible="no" active="yes"/>
+<layer number="117" name="mPads" color="7" fill="1" visible="no" active="yes"/>
 <layer number="118" name="Rect_Pads" color="7" fill="1" visible="no" active="yes"/>
+<layer number="119" name="mUnrouted" color="7" fill="1" visible="no" active="yes"/>
+<layer number="120" name="mDimension" color="7" fill="1" visible="no" active="yes"/>
 <layer number="121" name="_tsilk" color="7" fill="1" visible="no" active="yes"/>
 <layer number="122" name="_bsilk" color="7" fill="1" visible="no" active="yes"/>
@@
 <layer number="131" name="tAdjust" color="7" fill="1" visible="no" active="yes"/>
 <layer number="132" name="bAdjust" color="7" fill="1" visible="no" active="yes"/>
+<layer number="133" name="mtFinish" color="7" fill="1" visible="no" active="yes"/>
+<layer number="134" name="mbFinish" color="7" fill="1" visible="no" active="yes"/>
+<layer number="135" name="mtGlue" color="7" fill="1" visible="no" active="yes"/>
+<layer number="136" name="mbGlue" color="7" fill="1" visible="no" active="yes"/>
+<layer number="137" name="mtTest" color="7" fill="1" visible="no" active="yes"/>
+<layer number="138" name="mbTest" color="7" fill="1" visible="no" active="yes"/>
+<layer number="139" name="mtKeepout" color="7" fill="1" visible="no" active="yes"/>
+<layer number="140" name="mbKeepout" color="7" fill="1" visible="no" active="yes"/>
+<layer number="141" name="mtRestrict" color="7" fill="1" visible="no" active="yes"/>
+<layer number="142" name="mbRestrict" color="7" fill="1" visible="no" active="yes"/>
+<layer number="143" name="mvRestrict" color="7" fill="1" visible="no" active="yes"/>
 <layer number="144" name="Drill_legend" color="7" fill="1" visible="no" active="yes"/>
+<layer number="145" name="mHoles" color="7" fill="1" visible="no" active="yes"/>
+<layer number="146" name="mMilling" color="7" fill="1" visible="no" active="yes"/>
+<layer number="147" name="mMeasures" color="7" fill="1" visible="no" active="yes"/>
+<layer number="148" name="mDocument" color="7" fill="1" visible="no" active="yes"/>
+<layer number="149" name="mReference" color="7" fill="1" visible="no" active="yes"/>
 <layer number="150" name="Notes" color="7" fill="1" visible="no" active="yes"/>
 <layer number="151" name="HeatSink" color="7" fill="1" visible="no" active="yes"/>
@@
 <layer number="154" name="FabDoc2" color="7" fill="1" visible="no" active="yes"/>
 <layer number="155" name="FabDoc3" color="7" fill="1" visible="no" active="yes"/>
+<layer number="191" name="mNets" color="7" fill="1" visible="no" active="yes"/>
+<layer number="192" name="mBusses" color="7" fill="1" visible="no" active="yes"/>
+<layer number="193" name="mPins" color="7" fill="1" visible="no" active="yes"/>
+<layer number="194" name="mSymbols" color="7" fill="1" visible="no" active="yes"/>
 <layer number="195" name="ARDUINO_PIN_DESCRIPTION" color="7" fill="1" visible="no" active="yes"/>
 <layer number="196" name="ARDUINO_DIMENSION" color="7" fill="1" visible="no" active="yes"/>
@@
 <attribute name="VALUE" x="11.43" y="13.97" size="1.27" layer="28" rot="MR270"/>
 </element>
-<element name="CON" library="pinhead" library_urn="urn:adsk.eagle:library:325" package="1X04" package3d_urn="urn:adsk.eagle:package:22407/2" value="" x="54.61" y="12.7" smashed="yes" rot="R270">
-<attribute name="NAME" x="56.4388" y="17.8562" size="1.27" layer="25" ratio="10" rot="R270"/>
-<attribute name="POPULARITY" value="91" x="45.72" y="-13.97" size="1.778" layer="27" rot="R270" display="off"/>
-<attribute name="VALUE" x="51.435" y="17.78" size="1.27" layer="27" rot="R270"/>
-</element>
 <element name="D1" library="Wurth_Elektronik_Optoelectronics_rev15b" package="3528-2PIN" value="" x="49.53" y="12.7" smashed="yes" rot="R90">
 <attribute name="COMPANY-URL" value="http://www.we-online.de" x="52.07" y="29.21" size="1.778" layer="27" rot="R90" display="off"/>
@@
 <attribute name="VALUE" x="22.225" y="7.112" size="1.27" layer="28" rot="MR0"/>
 </element>
+<element name="MULTI2" library="CONNECTER" package="2.0_1X4" value="TWIG_2.0" x="54.61" y="12.7" smashed="yes" rot="MR270">
+<attribute name="NAME" x="52.029" y="17.637" size="0.8128" layer="26" font="vector" ratio="10" rot="MR270"/>
+<attribute name="NAME" x="53.81" y="17.5" size="0.8128" layer="34" font="vector" ratio="10" rot="MR270"/>
+</element>
 </elements>
 <signals>
@@
 <contactref element="Q4" pad="1"/>
 <contactref element="C3" pad="1"/>
-<contactref element="CON" pad="1"/>
 <contactref element="R1" pad="2"/>
 <contactref element="R4" pad="2"/>
 <contactref element="R3" pad="2"/>
 <contactref element="R2" pad="2"/>
-<wire x1="54.61" y1="16.51" x2="52.705" y2="16.51" width="0.508" layer="1"/>
-<wire x1="52.705" y1="16.51" x2="48.895" y2="20.32" width="0.508" layer="1"/>
+<wire x1="48.895" y1="20.32" x2="52.705" y2="16.51" width="0.508" layer="1"/>
 <wire x1="48.895" y1="20.32" x2="43.18" y2="20.32" width="0.508" layer="1"/>
 <wire x1="43.18" y1="20.32" x2="30.48" y2="20.32" width="0.508" layer="1"/>
@@
 <wire x1="46.04" y1="18.415" x2="46.04" y2="16.576" width="0.4064" layer="16"/>
 <wire x1="46.04" y1="16.576" x2="45.974" y2="16.51" width="0.4064" layer="16"/>
+<contactref element="MULTI2" pad="1"/>
+<wire x1="52.705" y1="16.51" x2="53.515" y2="15.7" width="0.508" layer="1"/>
+<wire x1="53.515" y1="15.7" x2="54.61" y2="15.7" width="0.508" layer="1"/>
 </signal>
 <signal name="GND">
@@
 <contactref element="C3" pad="2"/>
 <contactref element="C4" pad="2"/>
-<contactref element="CON" pad="4"/>
 <contactref element="D1" pad="1"/>
 <contactref element="D2" pad="1"/>
@@
 <vertex x="8.128" y="12.446"/>
 <vertex x="50.546" y="12.446"/>
-<vertex x="50.8" y="12.192"/>
-<vertex x="50.8" y="9.652"/>
-<vertex x="51.054" y="9.398"/>
-<vertex x="52.578" y="9.398"/>
-<vertex x="52.578" y="8.382"/>
+<vertex x="52.578" y="10.414"/>
+<vertex x="55.118" y="10.414"/>
+<vertex x="55.118" y="8.382"/>
 <vertex x="8.382" y="8.382"/>
 <vertex x="8.128" y="8.636"/>
-</polygon>
-<polygon width="0.0254" layer="16" thermals="no">
-<vertex x="54.61" y="9.398"/>
-<vertex x="52.324" y="9.398"/>
-<vertex x="52.324" y="8.382"/>
-<vertex x="54.61" y="8.382"/>
 </polygon>
 <wire x1="11.43" y1="11.275" x2="11.43" y2="9.525" width="0.4064" layer="1"/>
@@
 <wire x1="49.53" y1="11.275" x2="49.53" y2="9.525" width="0.4064" layer="1"/>
 <via x="49.53" y="9.525" extent="1-16" drill="0.35"/>
+<contactref element="MULTI2" pad="4"/>
 </signal>
 <signal name="SIG1">
@@
 <contactref element="R5" pad="2"/>
 <contactref element="Q2" pad="2"/>
-<contactref element="CON" pad="2"/>
 <wire x1="30.48" y1="10.8" x2="30.48" y2="12.192" width="0.3048" layer="1"/>
 <wire x1="30.988" y1="12.7" x2="30.48" y2="12.192" width="0.3048" layer="1"/>
-<wire x1="52.578" y1="13.97" x2="51.308" y2="12.7" width="0.3048" layer="1"/>
-<wire x1="54.61" y1="13.97" x2="52.578" y2="13.97" width="0.3048" layer="1"/>
 <wire x1="51.308" y1="12.7" x2="43.18" y2="12.7" width="0.3048" layer="1"/>
 <wire x1="43.18" y1="12.7" x2="30.988" y2="12.7" width="0.3048" layer="1"/>
@@
 <wire x1="43.434" y1="9.652" x2="43.18" y2="9.906" width="0.3048" layer="1"/>
 <wire x1="43.18" y1="9.906" x2="43.18" y2="10.8" width="0.3048" layer="1"/>
+<contactref element="MULTI2" pad="2"/>
+<wire x1="54.61" y1="13.7" x2="52.308" y2="13.7" width="0.3048" layer="1"/>
+<wire x1="52.308" y1="13.7" x2="51.308" y2="12.7" width="0.3048" layer="1"/>
 </signal>
 <signal name="SIG2">
@@
 <contactref element="R6" pad="2"/>
 <contactref element="Q4" pad="2"/>
-<contactref element="CON" pad="3"/>
 <wire x1="5.08" y1="10.8" x2="5.08" y2="12.192" width="0.3048" layer="1"/>
 <wire x1="5.08" y1="12.192" x2="5.588" y2="12.7" width="0.3048" layer="1"/>
@@
 <via x="19.05" y="9.652" extent="1-16" drill="0.35"/>
 <wire x1="19.05" y1="9.652" x2="17.78" y2="9.652" width="0.3048" layer="1"/>
-<wire x1="49.784" y1="8.382" x2="52.832" y2="11.43" width="0.3048" layer="1"/>
-<wire x1="52.832" y1="11.43" x2="54.61" y2="11.43" width="0.3048" layer="1"/>
-<wire x1="17.78" y1="8.382" x2="49.784" y2="8.382" width="0.3048" layer="1"/>
+<wire x1="49.784" y1="8.382" x2="17.78" y2="8.382" width="0.3048" layer="1"/>
+<contactref element="MULTI2" pad="3"/>
+<wire x1="54.61" y1="11.7" x2="53.102" y2="11.7" width="0.3048" layer="1"/>
+<wire x1="53.102" y1="11.7" x2="49.784" y2="8.382" width="0.3048" layer="1"/>
 </signal>
 <signal name="N$1">
