File: Eagle/Line sensors 2020/Line sensors - 6/Line sensors - 6.brd (EAGLE design)
At the start: 81.1 x 21 mm, 27 parts, among them Q1 VEMT2520X01, Q2 VEMT2520X01, Q3 VEMT2520X01, Q4 VEMT2520X01, Q5 VEMT2520X01, Q6 VEMT2520X01

Commit message: Final commit
Parts:
- removed CON: (no value), pinhead:1X04
- added MULTI2: TWIG_2.0, CONNECTER:2.0_1X4
Connections:
- net GND: now also MULTI2.4; no longer CON.4
- net SIG1: now also MULTI2.2; no longer CON.2
- net SIG2: now also MULTI2.3; no longer CON.3
- net V+: now also MULTI2.1; no longer CON.1
Changed lines of the file:
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@@
 <layer number="59" name="tCarbon" color="7" fill="1" visible="no" active="no"/>
 <layer number="60" name="bCarbon" color="7" fill="1" visible="no" active="no"/>
+<layer number="61" name="stand" color="7" fill="1" visible="no" active="no"/>
 <layer number="88" name="SimResults" color="9" fill="1" visible="no" active="no"/>
 <layer number="89" name="SimProbes" color="9" fill="1" visible="no" active="no"/>
@@
 <layer number="115" name="ReferenceISLANDS" color="7" fill="1" visible="no" active="yes"/>
 <layer number="116" name="Patch_BOT" color="9" fill="4" visible="no" active="yes"/>
+<layer number="117" name="mPads" color="7" fill="1" visible="no" active="yes"/>
 <layer number="118" name="Rect_Pads" color="7" fill="1" visible="no" active="yes"/>
+<layer number="119" name="mUnrouted" color="7" fill="1" visible="no" active="yes"/>
+<layer number="120" name="mDimension" color="7" fill="1" visible="no" active="yes"/>
 <layer number="121" name="_tsilk" color="7" fill="1" visible="no" active="yes"/>
 <layer number="122" name="_bsilk" color="7" fill="1" visible="no" active="yes"/>
@@
 <layer number="131" name="tAdjust" color="7" fill="1" visible="no" active="yes"/>
 <layer number="132" name="bAdjust" color="7" fill="1" visible="no" active="yes"/>
+<layer number="133" name="mtFinish" color="7" fill="1" visible="no" active="yes"/>
+<layer number="134" name="mbFinish" color="7" fill="1" visible="no" active="yes"/>
+<layer number="135" name="mtGlue" color="7" fill="1" visible="no" active="yes"/>
+<layer number="136" name="mbGlue" color="7" fill="1" visible="no" active="yes"/>
+<layer number="137" name="mtTest" color="7" fill="1" visible="no" active="yes"/>
+<layer number="138" name="mbTest" color="7" fill="1" visible="no" active="yes"/>
+<layer number="139" name="mtKeepout" color="7" fill="1" visible="no" active="yes"/>
+<layer number="140" name="mbKeepout" color="7" fill="1" visible="no" active="yes"/>
+<layer number="141" name="mtRestrict" color="7" fill="1" visible="no" active="yes"/>
+<layer number="142" name="mbRestrict" color="7" fill="1" visible="no" active="yes"/>
+<layer number="143" name="mvRestrict" color="7" fill="1" visible="no" active="yes"/>
 <layer number="144" name="Drill_legend" color="7" fill="1" visible="no" active="yes"/>
+<layer number="145" name="mHoles" color="7" fill="1" visible="no" active="yes"/>
+<layer number="146" name="mMilling" color="7" fill="1" visible="no" active="yes"/>
+<layer number="147" name="mMeasures" color="7" fill="1" visible="no" active="yes"/>
+<layer number="148" name="mDocument" color="7" fill="1" visible="no" active="yes"/>
+<layer number="149" name="mReference" color="7" fill="1" visible="no" active="yes"/>
 <layer number="150" name="Notes" color="7" fill="1" visible="no" active="yes"/>
 <layer number="151" name="HeatSink" color="7" fill="1" visible="no" active="yes"/>
@@
 <layer number="154" name="FabDoc2" color="7" fill="1" visible="no" active="yes"/>
 <layer number="155" name="FabDoc3" color="7" fill="1" visible="no" active="yes"/>
+<layer number="191" name="mNets" color="7" fill="1" visible="no" active="yes"/>
+<layer number="192" name="mBusses" color="7" fill="1" visible="no" active="yes"/>
+<layer number="193" name="mPins" color="7" fill="1" visible="no" active="yes"/>
+<layer number="194" name="mSymbols" color="7" fill="1" visible="no" active="yes"/>
 <layer number="195" name="ARDUINO_PIN_DESCRIPTION" color="7" fill="1" visible="no" active="yes"/>
 <layer number="196" name="ARDUINO_DIMENSION" color="7" fill="1" visible="no" active="yes"/>
@@
 <attribute name="VALUE" x="8.89" y="11.43" size="1.27" layer="28" rot="MR270"/>
 </element>
-<element name="CON" library="pinhead" library_urn="urn:adsk.eagle:library:325" package="1X04" package3d_urn="urn:adsk.eagle:package:22407/2" value="" x="77.47" y="10.16" smashed="yes" rot="R270">
-<attribute name="NAME" x="79.2988" y="15.3162" size="1.27" layer="25" ratio="10" rot="R270"/>
-<attribute name="POPULARITY" value="91" x="68.58" y="-24.13" size="1.778" layer="27" rot="R270" display="off"/>
-<attribute name="VALUE" x="74.295" y="15.24" size="1.27" layer="27" rot="R270"/>
-</element>
 <element name="D1" library="Wurth_Elektronik_Optoelectronics_rev15b" package="3528-2PIN" value="" x="72.39" y="10.16" smashed="yes" rot="R90">
 <attribute name="COMPANY-URL" value="http://www.we-online.de" x="74.93" y="26.67" size="1.778" layer="27" rot="R90" display="off"/>
@@
 <attribute name="SPICEPREFIX" value="R" x="11.43" y="-28.448" size="1.778" layer="28" rot="MR0" display="off"/>
 <attribute name="VALUE" x="32.385" y="4.572" size="1.27" layer="28" rot="MR0"/>
+</element>
+<element name="MULTI2" library="CONNECTER" package="2.0_1X4" value="TWIG_2.0" x="77.47" y="10.16" smashed="yes" rot="MR270">
+<attribute name="NAME" x="74.889" y="15.097" size="0.8128" layer="26" font="vector" ratio="10" rot="MR270"/>
+<attribute name="NAME" x="76.67" y="14.96" size="0.8128" layer="34" font="vector" ratio="10" rot="MR270"/>
 </element>
 </elements>
@@
 <contactref element="C5" pad="1"/>
 <contactref element="Q6" pad="1"/>
-<contactref element="CON" pad="1"/>
-<wire x1="77.47" y1="13.97" x2="74.93" y2="13.97" width="0.508" layer="1"/>
 <wire x1="72.39" y1="16.51" x2="66.04" y2="16.51" width="0.508" layer="1"/>
 <wire x1="66.04" y1="16.51" x2="53.34" y2="16.51" width="0.508" layer="1"/>
@@
 <wire x1="2.54" y1="15.24" x2="2.54" y2="13.462" width="0.508" layer="1"/>
 <wire x1="2.54" y1="13.462" x2="2.54" y2="12.06" width="0.508" layer="1"/>
-<wire x1="74.93" y1="13.97" x2="72.39" y2="16.51" width="0.508" layer="1"/>
+<wire x1="72.39" y1="16.51" x2="74.93" y2="13.97" width="0.508" layer="1"/>
 <wire x1="15.24" y1="12.06" x2="15.24" y2="13.462" width="0.508" layer="1"/>
 <wire x1="15.24" y1="13.462" x2="15.24" y2="16.51" width="0.508" layer="1"/>
@@
 <wire x1="5.4" y1="15.24" x2="5.4" y2="13.528" width="0.4064" layer="16"/>
 <wire x1="5.4" y1="13.528" x2="5.334" y2="13.462" width="0.4064" layer="16"/>
+<contactref element="MULTI2" pad="1"/>
+<wire x1="74.93" y1="13.97" x2="75.74" y2="13.16" width="0.6096" layer="1"/>
+<wire x1="75.74" y1="13.16" x2="77.47" y2="13.16" width="0.6096" layer="1"/>
 </signal>
 <signal name="N$1">
@@
 <contactref element="C4" pad="2"/>
 <contactref element="C5" pad="2"/>
-<contactref element="CON" pad="4"/>
-<polygon width="0.0254" layer="16" thermals="no">
-<vertex x="75.184" y="6.858"/>
-<vertex x="77.47" y="6.858"/>
-<vertex x="77.47" y="5.842"/>
-<vertex x="75.184" y="5.842"/>
-</polygon>
 <wire x1="8.89" y1="8.735" x2="8.89" y2="7.112" width="0.3048" layer="1"/>
 <via x="8.89" y="7.112" extent="1-16" drill="0.35"/>
@@
 <vertex x="5.588" y="6.096"/>
 <vertex x="5.842" y="5.842"/>
-<vertex x="75.438" y="5.842"/>
-<vertex x="75.438" y="6.858"/>
-<vertex x="74.93" y="6.858"/>
-<vertex x="74.676" y="7.112"/>
-<vertex x="74.676" y="9.652"/>
-<vertex x="74.422" y="9.906"/>
+<vertex x="77.978" y="5.842"/>
+<vertex x="77.978" y="8.128"/>
+<vertex x="76.454" y="8.128"/>
+<vertex x="74.676" y="9.906"/>
 </polygon>
+<contactref element="MULTI2" pad="4"/>
 </signal>
 <signal name="SIG1">
@@
 <contactref element="Q3" pad="2"/>
 <contactref element="R7" pad="2"/>
-<contactref element="CON" pad="2"/>
-<wire x1="75.184" y1="11.43" x2="73.914" y2="10.16" width="0.3048" layer="1"/>
 <wire x1="73.914" y1="10.16" x2="66.04" y2="10.16" width="0.3048" layer="1"/>
 <wire x1="66.04" y1="10.16" x2="53.34" y2="10.16" width="0.3048" layer="1"/>
@@
 <wire x1="40.894" y1="10.16" x2="40.64" y2="9.906" width="0.3048" layer="1"/>
 <wire x1="40.64" y1="9.906" x2="40.64" y2="8.26" width="0.3048" layer="1"/>
-<wire x1="77.47" y1="11.43" x2="75.184" y2="11.43" width="0.3048" layer="1"/>
 <wire x1="53.34" y1="8.26" x2="53.34" y2="10.16" width="0.3048" layer="1"/>
 <wire x1="66.04" y1="8.26" x2="66.04" y2="10.16" width="0.3048" layer="1"/>
@@
 <via x="66.802" y="7.112" extent="1-16" drill="0.35"/>
 <wire x1="66.802" y1="7.112" x2="68.9" y2="7.112" width="0.3048" layer="16"/>
+<contactref element="MULTI2" pad="2"/>
+<wire x1="77.47" y1="11.16" x2="74.914" y2="11.16" width="0.3048" layer="1"/>
+<wire x1="74.914" y1="11.16" x2="73.914" y2="10.16" width="0.3048" layer="1"/>
 </signal>
 <signal name="SIG2">
@@
 <contactref element="Q6" pad="2"/>
 <contactref element="R8" pad="2"/>
-<contactref element="CON" pad="3"/>
 <wire x1="2.54" y1="8.26" x2="2.54" y2="9.906" width="0.3048" layer="1"/>
 <wire x1="2.54" y1="9.906" x2="2.794" y2="10.16" width="0.3048" layer="1"/>
 <wire x1="2.794" y1="10.16" x2="15.24" y2="10.16" width="0.3048" layer="1"/>
 <wire x1="15.24" y1="8.26" x2="15.24" y2="10.16" width="0.3048" layer="1"/>
-<wire x1="72.39" y1="5.588" x2="75.692" y2="8.89" width="0.3048" layer="1"/>
-<wire x1="75.692" y1="8.89" x2="77.47" y2="8.89" width="0.3048" layer="1"/>
 <wire x1="27.94" y1="5.588" x2="72.39" y2="5.588" width="0.3048" layer="1"/>
 <wire x1="15.24" y1="10.16" x2="22.86" y2="10.16" width="0.3048" layer="1"/>
@@
 <wire x1="27.94" y1="7.112" x2="27.94" y2="5.588" width="0.3048" layer="1"/>
 <wire x1="29.337" y1="7.112" x2="27.94" y2="7.112" width="0.3048" layer="1"/>
+<contactref element="MULTI2" pad="3"/>
+<wire x1="75.962" y1="9.16" x2="77.47" y2="9.16" width="0.3048" layer="1"/>
+<wire x1="72.39" y1="5.588" x2="75.962" y2="9.16" width="0.3048" layer="1"/>
 </signal>
 </signals>
